Commit message: feat: env success condition, urdf limit

File: raisimGymME491/env/envs/aliengo_jump/rsc/aliengo/aliengo.urdf (robot description, URDF)
Before this commit: robot aliengo_description, 19 links, 18 joints
Joints:
- joint FL_calf_joint: limit (none) -> lower=-2.4696 upper=-0.0262 effort=60.0 velocity=30.0
- joint FL_hip_joint: limit (none) -> lower=-1.5708 upper=1.5708 effort=60.0 velocity=30.0
- joint FL_thigh_joint: limit (none) -> lower=-6.2832 upper=6.2832 effort=60.0 velocity=30.0
- joint FR_calf_joint: limit (none) -> lower=-2.4696 upper=-0.0262 effort=60.0 velocity=30.0
- joint FR_hip_joint: limit (none) -> lower=-1.5708 upper=1.5708 effort=60.0 velocity=30.0
- joint FR_thigh_joint: limit (none) -> lower=-6.2832 upper=6.2832 effort=60.0 velocity=30.0
- joint RL_calf_joint: limit (none) -> lower=-2.4696 upper=-0.0262 effort=60.0 velocity=30.0
- joint RL_hip_joint: limit (none) -> lower=-1.5708 upper=1.5708 effort=60.0 velocity=30.0
- joint RL_thigh_joint: limit (none) -> lower=-6.2832 upper=6.2832 effort=60.0 velocity=30.0
- joint RR_calf_joint: limit (none) -> lower=-2.4696 upper=-0.0262 effort=60.0 velocity=30.0
- joint RR_hip_joint: limit (none) -> lower=-1.5708 upper=1.5708 effort=60.0 velocity=30.0
- joint RR_thigh_joint: limit (none) -> lower=-6.2832 upper=6.2832 effort=60.0 velocity=30.0
